File: hotendheater.kicad_sch (KiCad schematic)
At the start: 13 parts, among them J1 Conn_01x02_Pin, J2 Conn_01x02_Pin, J3 Conn_01x08_Socket, J4 Conn_01x02_Pin, J5 Conn_01x02_Pin, Q1 IRF540N

Commit message: Improvements
Parts:
- removed J2: Conn_01x02_Pin, Connector_JST:JST_GH_BM02B-GHS-TBT_1x02-1MP_P1.25mm_Vertical, symbol Connector:Conn_01x02_Pin
- added H5, H6: MountingHole, MountingHole:MountingHole_3.2mm_M3_DIN965, symbol Mechanical:MountingHole
- added J6: Conn_01x02_Shielded, Connector_JST:JST_GH_SM02B-GHS-TB_1x02-1MP_P1.25mm_Horizontal, symbol Connector_Generic_Shielded:Conn_01x02_Shielded
- added R3: 10k, Resistor_SMD:R_0805_2012Metric, symbol Device:R
- J1: footprint Connector_JST:JST_XH_B2B-XH-AM_1x02_P2.50mm_Vertical -> Connector_JST:JST_XH_S2B-XH-A_1x02_P2.50mm_Horizontal
Connections:
- net GND: now also J6.2 (Pin_2), J6.SH (Shield), R3.1
- net Thermistor: now also J6.1 (Pin_1)
- net at Q1.1 (G), R1.2: now also R3.2
